File: UltrasoundDriver.kicad_sch (KiCad schematic)
At the start: 20 parts, among them J1 Conn_01x05_Female, J2 Conn_01x05_Female, U1 MC33079, U2 L7815, U3 L7915, U4 MC33079

Commit message: this draft has gone to justin
Parts:
- removed D1, D2: 1N4001, Diode_THT:D_DO-41_SOD81_P10.16mm_Horizontal, symbol Diode:1N4001
- added D1, D2: 1N4148W, Diode_SMD:D_SOD-123, symbol Diode:1N4148W
- C11, C12, C5, C6: footprint Capacitor_SMD:C_0603_1608Metric -> Capacitor_Tantalum_SMD:CP_EIA-3216-18_Kemet-A
Connections:
- net +15V: now also D1.1 (K)
- net -15V: now also D2.2 (A)
- net GND: now also D1.2 (A), D2.1 (K)
Changed lines of the file:
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@@
       (effects (font (size 1.27 1.27)) (justify left))
     )
-    (property "Footprint" "Capacitor_SMD:C_0603_1608Metric" (id 2) (at 109.22 43.18 0)
+    (property "Footprint" "Capacitor_Tantalum_SMD:CP_EIA-3216-18_Kemet-A" (id 2) (at 109.22 43.18 0)
       (effects (font (size 1.27 1.27)) hide)
     )
@@
       (effects (font (size 1.27 1.27)) (justify left))
     )
-    (property "Footprint" "Capacitor_SMD:C_0603_1608Metric" (id 2) (at 109.22 55.88 0)
+    (property "Footprint" "Capacitor_Tantalum_SMD:CP_EIA-3216-18_Kemet-A" (id 2) (at 109.22 55.88 0)
       (effects (font (size 1.27 1.27)) hide)
     )
@@
       (effects (font (size 1.27 1.27)) (justify left))
     )
-    (property "Footprint" "Capacitor_SMD:C_0603_1608Metric" (id 2) (at 139.7 43.18 0)
+    (property "Footprint" "Capacitor_Tantalum_SMD:CP_EIA-3216-18_Kemet-A" (id 2) (at 139.7 43.18 0)
       (effects (font (size 1.27 1.27)) hide)
     )
@@
       (effects (font (size 1.27 1.27)) (justify left))
     )
-    (property "Footprint" "Capacitor_SMD:C_0603_1608Metric" (id 2) (at 139.7 55.88 0)
+    (property "Footprint" "Capacitor_Tantalum_SMD:CP_EIA-3216-18_Kemet-A" (id 2) (at 139.7 55.88 0)
       (effects (font (size 1.27 1.27)) hide)
     )
     (property "Datasheet" "~" (id 3) (at 139.7 55.88 0)
-      (effects (font (size 1.27 1.27)) hide)
-    )
-    (pin "1")
-    (pin "2")
-  )
-  (symbol (lib_id "Diode:1N4001") (at 151.13 43.18 270) (unit 1)
-    (in_bom yes) (on_board yes)
-    (property "Reference" "D1" (id 0) (at 153.1366 42.0116 90)
-      (effects (font (size 1.27 1.27)) (justify left))
-    )
-    (property "Value" "1N4001" (id 1) (at 153.1366 44.323 90)
-      (effects (font (size 1.27 1.27)) (justify left))
-    )
-    (property "Footprint" "Diode_THT:D_DO-41_SOD81_P10.16mm_Horizontal" (id 2) (at 146.685 43.18 0)
-      (effects (font (size 1.27 1.27)) hide)
-    )
-    (property "Datasheet" "http://www.vishay.com/docs/88503/1n4001.pdf" (id 3) (at 151.13 43.18 0)
-      (effects (font (size 1.27 1.27)) hide)
-    )
-    (pin "1")
-    (pin "2")
-  )
-  (symbol (lib_id "Diode:1N4001") (at 151.13 55.88 270) (unit 1)
-    (in_bom yes) (on_board yes)
-    (property "Reference" "D2" (id 0) (at 153.1366 54.7116 90)
-      (effects (font (size 1.27 1.27)) (justify left))
-    )
-    (property "Value" "1N4001" (id 1) (at 153.1366 57.023 90)
-      (effects (font (size 1.27 1.27)) (justify left))
-    )
-    (property "Footprint" "Diode_THT:D_DO-41_SOD81_P10.16mm_Horizontal" (id 2) (at 146.685 55.88 0)
-      (effects (font (size 1.27 1.27)) hide)
-    )
-    (property "Datasheet" "http://www.vishay.com/docs/88503/1n4001.pdf" (id 3) (at 151.13 55.88 0)
       (effects (font (size 1.27 1.27)) hide)
     )
@@
     (pin "2")
   )
+  (symbol (lib_id "Diode:1N4148W") (at 151.13 43.18 270) (unit 1)
+    (in_bom yes) (on_board yes) (fields_autoplaced)
+    (property "Reference" "D1" (id 0) (at 153.162 42.3453 90)
+      (effects (font (size 1.27 1.27)) (justify left))
+    )
+    (property "Value" "1N4148W" (id 1) (at 153.162 44.8822 90)
+      (effects (font (size 1.27 1.27)) (justify left))
+    )
+    (property "Footprint" "Diode_SMD:D_SOD-123" (id 2) (at 146.685 43.18 0)
+      (effects (font (size 1.27 1.27)) hide)
+    )
+    (property "Datasheet" "https://www.vishay.com/docs/85748/1n4148w.pdf" (id 3) (at 151.13 43.18 0)
+      (effects (font (size 1.27 1.27)) hide)
+    )
+    (pin "1")
+    (pin "2")
+  )
+  (symbol (lib_id "Diode:1N4148W") (at 151.13 55.88 270) (unit 1)
+    (in_bom yes) (on_board yes) (fields_autoplaced)
+    (property "Reference" "D2" (id 0) (at 153.162 55.0453 90)
+      (effects (font (size 1.27 1.27)) (justify left))
+    )
+    (property "Value" "1N4148W" (id 1) (at 153.162 57.5822 90)
+      (effects (font (size 1.27 1.27)) (justify left))
+    )
+    (property "Footprint" "Diode_SMD:D_SOD-123" (id 2) (at 146.685 55.88 0)
+      (effects (font (size 1.27 1.27)) hide)
+    )
+    (property "Datasheet" "https://www.vishay.com/docs/85748/1n4148w.pdf" (id 3) (at 151.13 55.88 0)
+      (effects (font (size 1.27 1.27)) hide)
+    )
+    (pin "1")
+    (pin "2")
+  )
   (sheet (at 34.29 129.54) (size 33.02 24.13) (fields_autoplaced)
     (stroke (width 0) (type solid) (color 0 0 0 0))
@@
     )
     (path "/00000000-0000-0000-0000-0000633337cc"
-      (reference "C5") (unit 1) (value "0.33u") (footprint "Capacitor_SMD:C_0603_1608Metric")
+      (reference "C5") (unit 1) (value "0.33u") (footprint "Capacitor_Tantalum_SMD:CP_EIA-3216-18_Kemet-A")
     )
     (path "/00000000-0000-0000-0000-000063334f88"
-      (reference "C6") (unit 1) (value "2.2u") (footprint "Capacitor_SMD:C_0603_1608Metric")
+      (reference "C6") (unit 1) (value "2.2u") (footprint "Capacitor_Tantalum_SMD:CP_EIA-3216-18_Kemet-A")
     )
     (path "/00000000-0000-0000-0000-00006337fda0"
@@
     )
     (path "/00000000-0000-0000-0000-000063338a2a"
-      (reference "C11") (unit 1) (value "0.1u") (footprint "Capacitor_SMD:C_0603_1608Metric")
+      (reference "C11") (unit 1) (value "0.1u") (footprint "Capacitor_Tantalum_SMD:CP_EIA-3216-18_Kemet-A")
     )
     (path "/00000000-0000-0000-0000-00006333930a"
-      (reference "C12") (unit 1) (value "1u") (footprint "Capacitor_SMD:C_0603_1608Metric")
+      (reference "C12") (unit 1) (value "1u") (footprint "Capacitor_Tantalum_SMD:CP_EIA-3216-18_Kemet-A")
     )
     (path "/00000000-0000-0000-0000-00006310453c/00000000-0000-0000-0000-000063113f14"
@@
       (reference "C16") (unit 1) (value "100n") (footprint "Capacitor_SMD:C_0603_1608Metric")
     )
-    (path "/00000000-0000-0000-0000-000063339f89"
-      (reference "D1") (unit 1) (value "1N4001") (footprint "Diode_THT:D_DO-41_SOD81_P10.16mm_Horizontal")
-    )
-    (path "/00000000-0000-0000-0000-00006333baf3"
-      (reference "D2") (unit 1) (value "1N4001") (footprint "Diode_THT:D_DO-41_SOD81_P10.16mm_Horizontal")
-    )
-    (path "/00000000-0000-0000-0000-00006310453c/00000000-0000-0000-0000-00006311b215"
-      (reference "D3") (unit 1) (value "1N914") (footprint "Diode_THT:D_DO-35_SOD27_P7.62mm_Horizontal")
-    )
-    (path "/00000000-0000-0000-0000-00006310453c/00000000-0000-0000-0000-00006311d65a"
-      (reference "D4") (unit 1) (value "1N914") (footprint "Diode_THT:D_DO-35_SOD27_P7.62mm_Horizontal")
-    )
-    (path "/00000000-0000-0000-0000-000063143e55/00000000-0000-0000-0000-00006339677d"
-      (reference "D5") (unit 1) (value "1N5819") (footprint "Diode_THT:D_DO-41_SOD81_P10.16mm_Horizontal")
-    )
-    (path "/00000000-0000-0000-0000-000063143e55/00000000-0000-0000-0000-000063399fc8"
-      (reference "D6") (unit 1) (value "1N5819") (footprint "Diode_THT:D_DO-41_SOD81_P10.16mm_Horizontal")
+    (path "/705400fa-62b9-42be-acd7-36640e652531"
+      (reference "D1") (unit 1) (value "1N4148W") (footprint "Diode_SMD:D_SOD-123")
+    )
+    (path "/99aa5e43-e983-4d95-b358-514ef420a0fa"
+      (reference "D2") (unit 1) (value "1N4148W") (footprint "Diode_SMD:D_SOD-123")
+    )
+    (path "/00000000-0000-0000-0000-00006310453c/2885c455-af22-48fb-b03e-5779fc306315"
+      (reference "D3") (unit 1) (value "1N4148W") (footprint "Diode_SMD:D_SOD-123")
+    )
+    (path "/00000000-0000-0000-0000-00006310453c/8d057da6-c621-49d8-8c9c-1a79a55a84a2"
+      (reference "D4") (unit 1) (value "1N4148W") (footprint "Diode_SMD:D_SOD-123")
+    )
+    (path "/00000000-0000-0000-0000-000063143e55/9ae8eb7e-9653-49f7-b132-205d6381d0c1"
+      (reference "D5") (unit 1) (value "B5819W.SL") (footprint "SamacSys_Parts:B5819WSL")
+    )
+    (path "/00000000-0000-0000-0000-000063143e55/858c5b99-a8d5-44e4-8242-15bcd1a0ce5f"
+      (reference "D6") (unit 1) (value "B5819W.SL") (footprint "SamacSys_Parts:B5819WSL")
     )
     (path "/00000000-0000-0000-0000-0000630cd5ba"
@@
       (reference "LS2") (unit 1) (value "400ST16M") (footprint "SamacSys_Parts:400ST16M")
     )
-    (path "/00000000-0000-0000-0000-00006310453c/00000000-0000-0000-0000-00006310a68f"
-      (reference "Q1") (unit 1) (value "S8050") (footprint "Package_TO_SOT_THT:TO-92_Inline")
-    )
-    (path "/00000000-0000-0000-0000-00006310453c/00000000-0000-0000-0000-00006310a695"
-      (reference "Q2") (unit 1) (value "S8550") (footprint "Package_TO_SOT_THT:TO-92_Inline")
+    (path "/00000000-0000-0000-0000-00006310453c/6771dd30-6316-4928-ae16-a4fab88a526b"
+      (reference "Q1") (unit 1) (value "SS8050-G") (footprint "SamacSys_Parts:SOT95P240X115-3N")
+    )
+    (path "/00000000-0000-0000-0000-00006310453c/eaef602c-0099-4f05-b952-25b2bc19c63f"
+      (reference "Q2") (unit 1) (value "S8550") (footprint "SamacSys_Parts:SOT95P240X115-3N")
     )
     (path "/00000000-0000-0000-0000-00006310453c/00000000-0000-0000-0000-0000631109af"
@@
     )
     (path "/00000000-0000-0000-0000-00006310453c/00000000-0000-0000-0000-000063119e7e"
-      (reference "R4") (unit 1) (value "5.8k") (footprint "Resistor_SMD:R_0603_1608Metric")
+      (reference "R4") (unit 1) (value "6.8k") (footprint "Resistor_SMD:R_0603_1608Metric")
     )
     (path "/00000000-0000-0000-0000-00006310453c/00000000-0000-0000-0000-000063119e84"
