File: outputDriver.kicad_sch (KiCad schematic)
At the start: 16 parts, among them Q1 S8050, Q2 S8550, U1 MC33079

Commit message: yeah I think this one is better, also updated resistor values after lab work
Parts:
- R4: value 4.7k -> 5.8k
Changed lines of the file:
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@@
       (effects (font (size 1.27 1.27)) (justify left))
     )
-    (property "Value" "4.7k" (id 1) (at 160.4772 88.773 0)
+    (property "Value" "5.8k" (id 1) (at 160.4772 88.773 0)
       (effects (font (size 1.27 1.27)) (justify left))
     )

Commit message: this draft has gone to justin
Parts:
- removed D3, D4: 1N914, Diode_THT:D_DO-35_SOD27_P7.62mm_Horizontal, symbol Diode:1N914
- removed Q1: S8050, Package_TO_SOT_THT:TO-92_Inline, symbol Transistor_BJT:S8050
- removed Q2: S8550, Package_TO_SOT_THT:TO-92_Inline, symbol Transistor_BJT:S8550
- added D3, D4: 1N4148W, Diode_SMD:D_SOD-123, symbol Diode:1N4148W
- added Q1: SS8050-G, SamacSys_Parts:SOT95P240X115-3N, symbol SamacSys_Parts:SS8050-G
- added Q2: S8550, SamacSys_Parts:SOT95P240X115-3N, symbol SamacSys_Parts:S8550
- R4: value 5.8k -> 6.8k
Connections:
- net +15V: now also Q1.3
- net -15V: now also Q2.3
- net at U1.7: now also D3.1 (K), D4.2 (A)
- net at R8.1: now also Q1.2
- net at R6.2: now also D3.2 (A), Q1.1
- net at R9.1: now also Q2.2
- net at R7.1: now also D4.1 (K), Q2.1

Commit message: updated and sent to Justin
Connections:
- net at C13.1, R3.2: now also U1.12 (+); no longer U1.5 (+)
- net at R4.2, R5.1: now also U1.13 (-); no longer U1.6 (-)
- net at D3.1 (K), D4.2 (A): now also U1.14; no longer U1.7
Changed lines of the file:
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@@
     (pin "4")
   )
-  (symbol (lib_id "Amplifier_Operational:MC33079") (at 151.13 74.93 0) (unit 2)
+  (symbol (lib_id "Amplifier_Operational:MC33079") (at 151.13 74.93 0) (unit 4)
     (in_bom yes) (on_board yes)
     (property "Reference" "U1" (id 0) (at 151.13 65.6082 0))
